File: PCB/motionalr_mcu.kicad_pcb (KiCad board)
At the start: 2 copper layers, 47.6 x 50 mm, 11 parts, among them J1 J1_SENSOR, Q1 2N222, U1 XIAO-ESP32-C3-DIP

Commit message: Changed a typo in schematics
Other:
- board text added: "1-3V3 2-GND 3-OT2 4-RX 5-TX"
- board text removed: "1-3V3 2-GND 3-OT2 4-TX 5-RX"
Changed lines of the file:
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@@
 		)
 	)
-	(gr_text "1-3V3\n2-GND\n3-OT2\n4-TX\n5-RX"
+	(gr_text "1-3V3\n2-GND\n3-OT2\n4-RX\n5-TX"
 		(at 147.6375 88.10625 0)
 		(layer "F.SilkS")
