File: PCB/motionalr_mcu.kicad_sch (KiCad schematic)
At the start: 11 parts, among them J1 J1_SENSOR, Q1 2N222, U1 XIAO-ESP32-C3-DIP

Commit message: Changed a typo in schematics
Connections:
- net RX: now also J1.4 (Pin_4), R5.2; no longer J1.5 (Pin_5), R4.2
- net TX: now also J1.5 (Pin_5), R4.2; no longer J1.4 (Pin_4), R5.2
Changed lines of the file:
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@@
 		)
 	)
-	(label "TX"
+	(label "RX"
 		(at 162.56 64.77 0)
 		(effects
@@
 		)
 	)
-	(label "RX"
+	(label "TX"
 		(at 166.37 67.31 0)
 		(effects
